Commit message: updated urdf to work with the current code

File: urdf/track_collision.urdf.xacro (robot description, xacro)
@@ -38,5 +38,5 @@
       <origin xyz="${xyz}" rpy="${rpy}" />
     </joint>
-    <gazebo reference="{name}_link">
+    <gazebo reference="${name}_link">
       <selfCollide>false</selfCollide>
       <static>false</static>

File: urdf/trailblazer.urdf.xacro (robot description, xacro)
@@ -11,5 +11,5 @@
   <!-- Load calibration -->
   <xacro:include filename="$(find trailblazer_description)/urdf/tools/calibration.urdf.xacro" />
-  <xacro:property name="calibration" value="${load_yaml('$(find trailblazer_description)/config/calibration.yaml')}" />
+  <xacro:property name="calibration" value="${xacro.load_yaml('$(find trailblazer_description)/config/calibration.yaml')}" />
   <!-- Add sensors: IMU -->
   <link name="xsens_imu_link"/>
